File: KiCad/C3/Unified-Daughterboard.kicad_sch (KiCad schematic)
At the start: 11 parts

Commit message: Trimmer version
Parts:
- UMH1: footprint nopun-keyboard-parts:leopold_db_outline -> nopun-keyboard-parts:leopold_db_trimmer
- gave numbers to parts that had none: 8
Changed lines of the file:
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@@
   (symbol (lib_id "Connector_Generic:Conn_01x04") (at 241.3 77.47 0) (unit 1)
     (in_bom yes) (on_board yes)
-    (property "Reference" "" (id 0) (at 243.84 74.93 0)
+    (property "Reference" "J2" (id 0) (at 243.84 74.93 0)
       (effects (font (size 1.27 1.27)) (justify left))
     )
@@
   (symbol (lib_id "Device:R_Small") (at 59.055 42.545 90) (unit 1)
     (in_bom yes) (on_board yes)
-    (property "Reference" "" (id 0) (at 59.055 40.64 90)
+    (property "Reference" "R1" (id 0) (at 59.055 40.64 90)
       (effects (font (size 0.762 0.762)))
     )
@@
   (symbol (lib_id "Device:R_Small") (at 59.055 47.625 90) (unit 1)
     (in_bom yes) (on_board yes)
-    (property "Reference" "" (id 0) (at 59.055 45.72 90)
+    (property "Reference" "R2" (id 0) (at 59.055 45.72 90)
       (effects (font (size 0.762 0.762)))
     )
@@
   (symbol (lib_id "Device:D_TVS") (at 113.665 90.17 270) (mirror x) (unit 1)
     (in_bom yes) (on_board yes)
-    (property "Reference" "" (id 0) (at 109.855 90.17 0)
+    (property "Reference" "D1" (id 0) (at 109.855 90.17 0)
       (effects (font (size 0.762 0.762)))
     )
@@
   (symbol (lib_id "acheronSymbols:TYPE-C-31-M12_13") (at 40.005 59.055 0) (unit 1)
     (in_bom yes) (on_board yes)
-    (property "Reference" "" (id 0) (at 40.005 22.86 0))
+    (property "Reference" "J1" (id 0) (at 40.005 22.86 0))
     (property "Value" "TYPE-C-31-M12_13" (id 1) (at 40.005 25.4 0))
     (property "Footprint" "acheron_Connectors:TYPE-C-31-M-12" (id 2) (at 27.305 57.785 90)
@@
   (symbol (lib_id "acheronSymbols:TPD4E05U06DQAR") (at 111.125 43.815 0) (unit 1)
     (in_bom yes) (on_board yes)
-    (property "Reference" "" (id 0) (at 111.125 31.9786 0))
+    (property "Reference" "U1" (id 0) (at 111.125 31.9786 0))
     (property "Value" "TPD4E05U06DQAR" (id 1) (at 111.125 34.29 0))
     (property "Footprint" "acheron_Components:USON-10_2.5x1.0mm_P0.5mm" (id 2) (at 111.125 17.145 0)
@@
   (symbol (lib_id "Device:Polyfuse") (at 107.315 85.09 90) (unit 1)
     (in_bom yes) (on_board yes)
-    (property "Reference" "" (id 0) (at 107.315 80.645 90))
+    (property "Reference" "F1" (id 0) (at 107.315 80.645 90))
     (property "Value" "ASMD1206-150" (id 1) (at 107.315 82.3214 90)
       (effects (font (size 0.508 0.508)))
@@
   (symbol (lib_id "Device:L_Ferrite") (at 32.385 114.935 0) (unit 1)
     (in_bom yes) (on_board yes)
-    (property "Reference" "" (id 0) (at 34.6202 113.792 0)
+    (property "Reference" "L1" (id 0) (at 34.6202 113.792 0)
       (effects (font (size 1.27 1.27)) (justify left))
     )
@@
       (effects (font (size 1.27 1.27)) (justify left))
     )
-    (property "Footprint" "nopun-keyboard-parts:leopold_db_outline" (id 2) (at 176.53 60.96 0)
+    (property "Footprint" "nopun-keyboard-parts:leopold_db_trimmer" (id 2) (at 176.53 60.96 0)
       (effects (font (size 1.27 1.27)) hide)
     )
@@
     )
     (path "/dfaa9fe6-4459-4ab5-b7b1-477247fdfc6e"
-      (reference "UMH1") (unit 1) (value "Outline") (footprint "nopun-keyboard-parts:leopold_db_outline")
-    )
-  )
+      (reference "UMH1") (unit 1) (value "Outline") (footprint "nopun-keyboard-parts:leopold_db_trimmer")
+    )
+  )
